File: design/usb.kicad_sch (KiCad schematic)
At the start: 8 parts, among them J2 USB_C_Receptacle, U3 TPS25750D

Commit message: LDOs
Changed lines of the file:
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@@
   (junction (at 136.525 47.625) (diameter 0) (color 0 0 0 0)
-  )
-  (junction (at 172.085 102.87) (diameter 0) (color 0 0 0 0)
   )
   (junction (at 136.525 64.77) (diameter 0) (color 0 0 0 0)
@@
     (stroke (width 0) (type default))
   )
-  (wire (pts (xy 171.45 102.87) (xy 172.085 102.87))
-    (stroke (width 0) (type default))
-  )
