File: design/pages/fpga.kicad_sch (KiCad schematic)
At the start: 0 parts

Commit message: USB PD
Parts:
- added U2: ICE40HX8K-BG121, Package_BGA:BGA-121_9.0x9.0mm_Layout11x11_P0.8mm_Ball0.4mm_Pad0.35mm_NSMD, symbol FPGA_Lattice:ICE40HX8K-BG121
Connections:
- new net: U2.D4 (VCC), U2.D8 (VCC), U2.H4 (VCC), U2.H8 (VCC)
- new net: U2.E5 (GND), U2.E6 (GND), U2.E7 (GND), U2.F5 (GND), U2.F6 (GND), U2.F7 (GND), U2.G5 (GND), U2.G6 (GND), U2.G7 (GND), U2.H5 (GND)
- new net: U2.E4 (VCCIO_3), U2.G4 (VCCIO_3)
