File: design/pages/mcu.kicad_sch (KiCad schematic)
At the start: 0 parts

Commit message: USB PD
Parts:
- added C1: 10uF, Capacitor_SMD:C_0402_1005Metric, symbol elias_kountouris_manifest:C_10uF_6.3V_0402
- added C2, C3, C4, C5, C6: 100nF, Capacitor_SMD:C_0402_1005Metric, symbol elias_kountouris_manifest:C_100nF_16V_0402
- added C7: 1uF, Capacitor_SMD:C_0402_1005Metric, symbol elias_kountouris_manifest:C_1uF_6.3V_0402
- added C8: 4.7uF, Capacitor_SMD:C_0402_1005Metric, symbol elias_kountouris_manifest:C_4.7_10V_0402
- added J1: 1x3 Pin, symbol Connector:Conn_01x03_Pin
- added R1: 100k, Resistor_SMD:R_0402_1005Metric, symbol elias_kountouris_manifest:R_100k_0402
- added U1: STM32F410C8Ux, Package_DFN_QFN:QFN-48-1EP_7x7mm_P0.5mm_EP5.6x5.6mm, symbol MCU_ST_STM32F4:STM32F410C8Ux
Connections:
- new net: R1.2, U1.7 (NRST)
- new net: J1.2 (Pin_2), U1.44 (BOOT0)
- new net: C8.1, U1.22 (VCAP1)
- new net +3.3V: C1.1, C2.1, C3.1, C4.1, C5.1, J1.1 (Pin_1), R1.1, U1.1 (VBAT), U1.24 (VDD), U1.36 (VDD), U1.48 (VDD)
- new net +3.3VA: C6.1, C7.1, U1.9 (VDDA)
- new net BOOTLOADER_USART_RX: U1.31 (PA10)
- new net BOOTLOADER_USART_TX: U1.30 (PA9)
- new net GND: C1.2, C2.2, C3.2, C4.2, C5.2, C6.2, C7.2, C8.2, J1.3 (Pin_3), U1.23 (VSS), U1.35 (VSS), U1.47 (VSS), U1.49 (VSS), U1.8 (VSSA)
- new net JNTRST: U1.40 (PB4)
- new net JTCK: U1.37 (PA14)
- new net JTDI: U1.38 (PA15)
- new net JTDO: U1.39 (PB3)
- new net JTMS: U1.34 (PA13)
Other:
- note added: "JTAG pins have some pullups / pulldowns on them even when in GPIO mode"
