File: design/pages/pmu.kicad_sch (KiCad schematic)
At the start: 0 parts

Commit message: LDOs
Parts:
- added C11, C12, C13, C14: 1uF, Capacitor_SMD:C_0402_1005Metric, symbol elias_kountouris_manifest:C_1uF_6.3V_0402
- added U4, U5: TLV74033, Package_TO_SOT_SMD:SOT-23-5, symbol oscilliscope:TLV74033
Connections:
- new net +3.3VA: C12.1, U4.5 (OUT)
- new net +3V3: C14.1, U5.5 (OUT)
- new net +5V: C11.1, C13.1, U4.1 (IN), U4.3 (EN), U5.1 (IN), U5.3 (EN)
- new net GND: C11.2, C12.2, C13.2, C14.2, U4.2 (GND), U5.2 (GND)
Other:
- note added: "Analog Power Budget: ADC1: 26mA ADC2: 26mA Total: Digital Power Budget: MCU: 10mA"
